File: STM32 Klipper Expander.kicad_pcb (KiCad board)
At the start: 2 copper layers, 44.4 x 44.5 mm, 28 parts, among them J1 Conn_01x04, J2 USB_B_Micro, J3 Conn_02x05, J4 Conn_01x03, J5 Screw_Terminal_01x08, Q1 IRLML6344TRPBF, Q2 IRLML6344TRPBF, Q3 IRLML6344TRPBF, Q4 IRLML6344TRPBF, SW1 SW_SPST, SW2 SW_SPST, U1 STM32F042F6Px, U2 AP2127K-3.3

Commit message: Initial Commit
Parts:
- moved J3 0.71 mm to (140.0, 58.7)
- moved J4 0.69 mm to (135.6, 59.4)
Changed lines of the file:
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@@
     (aux_axis_origin 0 0)
     (grid_origin 129.845 86.03)
-    (visible_elements FFFFFF7F)
+    (visible_elements 7FFFFFFF)
     (pcbplotparams
       (layerselection 0x010fc_ffffffff)
@@
   )
   (module Connector_PinHeader_2.54mm:PinHeader_1x03_P2.54mm_Vertical (layer F.Cu)
-    (at 135.595 58.67)
+    (at 135.56 59.36)
     (descr "Through hole straight pin header, 1x03, 2.54mm pitch, single row")
     (tags "Through hole pin header THT 1x03 2.54mm single row")
@@
   )
   (module Connector_PinHeader_1.27mm:PinHeader_2x05_P1.27mm_Vertical (layer F.Cu)
-    (at 140.045 58.02)
+    (at 140.005 58.725)
     (descr "Through hole straight pin header, 2x05, 1.27mm pitch, double rows")
     (tags "Through hole pin header THT 2x05 1.27mm double row")
@@
     (arrow2b (pts (xy 89.84 100) (xy 89.253579 98.873496)))
   )
-  (via (at 127.94 82.855) (size 0.8) (drill 0.4) (layers F.Cu B.Cu) (net 5))
   (segment (start 134.5215 83.8) (end 135.052 84.3305) (width 0.3) (layer F.Cu) (net 1))
   (segment (start 132.16 83.8) (end 134.5215 83.8) (width 0.3) (layer F.Cu) (net 1))
@@
   (segment (start 140.005 91.11) (end 140.005 86.885002) (width 0.25) (layer F.Cu) (net 3))
   (segment (start 118.415 95.8875) (end 118.415 93.9525) (width 0.25) (layer F.Cu) (net 4))
+  (via (at 127.94 82.855) (size 0.8) (drill 0.4) (layers F.Cu B.Cu) (net 5))
   (segment (start 127.94 87.935) (end 126.035 89.84) (width 0.25) (layer B.Cu) (net 5))
   (segment (start 127.585 82.5) (end 126.26 82.5) (width 0.25) (layer F.Cu) (net 5))
@@
   (segment (start 134.3725 81.2) (end 134.6225 80.95) (width 0.25) (layer F.Cu) (net 10))
   (segment (start 132.16 81.2) (end 134.3725 81.2) (width 0.25) (layer F.Cu) (net 10))
+  (segment (start 113.97 95.555) (end 114.605 94.92) (width 2) (layer F.Cu) (net 13))
+  (segment (start 105.715 95.555) (end 113.97 95.555) (width 2) (layer F.Cu) (net 13))
+  (segment (start 113.97 85.395) (end 114.605 84.76) (width 2) (layer F.Cu) (net 14))
+  (segment (start 105.715 85.395) (end 113.97 85.395) (width 2) (layer F.Cu) (net 14))
   (segment (start 113.97 75.235) (end 114.605 74.6) (width 2) (layer F.Cu) (net 15))
   (segment (start 105.715 75.235) (end 113.97 75.235) (width 2) (layer F.Cu) (net 15))
-  (segment (start 115.5425 72.9025) (end 115.555 72.915) (width 0.5) (layer F.Cu) (net 18))
-  (segment (start 115.5425 69.52) (end 115.5425 72.9025) (width 0.5) (layer F.Cu) (net 18))
-  (segment (start 113.97 85.395) (end 114.605 84.76) (width 2) (layer F.Cu) (net 14))
-  (segment (start 105.715 85.395) (end 113.97 85.395) (width 2) (layer F.Cu) (net 14))
-  (segment (start 115.5425 83.0625) (end 115.555 83.075) (width 0.5) (layer F.Cu) (net 19))
-  (segment (start 115.5425 79.68) (end 115.5425 83.0625) (width 0.5) (layer F.Cu) (net 19))
-  (segment (start 113.97 95.555) (end 114.605 94.92) (width 2) (layer F.Cu) (net 13))
-  (segment (start 105.715 95.555) (end 113.97 95.555) (width 2) (layer F.Cu) (net 13))
-  (segment (start 115.5425 93.2225) (end 115.555 93.235) (width 0.5) (layer F.Cu) (net 20))
-  (segment (start 115.5425 89.84) (end 115.5425 93.2225) (width 0.5) (layer F.Cu) (net 20))
   (segment (start 113.97 65.075) (end 114.605 64.44) (width 2) (layer F.Cu) (net 16))
   (segment (start 105.715 65.075) (end 113.97 65.075) (width 2) (layer F.Cu) (net 16))
@@
   (segment (start 119.05 65.075) (end 116.315 62.34) (width 0.25) (layer F.Cu) (net 17))
   (segment (start 119.05 83.49) (end 119.05 65.075) (width 0.25) (layer F.Cu) (net 17))
+  (segment (start 115.5425 72.9025) (end 115.555 72.915) (width 0.5) (layer F.Cu) (net 18))
+  (segment (start 115.5425 69.52) (end 115.5425 72.9025) (width 0.5) (layer F.Cu) (net 18))
   (segment (start 126.26 85.75) (end 120.04 85.75) (width 0.25) (layer F.Cu) (net 18))
   (segment (start 120.04 85.75) (end 118.415 84.125) (width 0.25) (layer F.Cu) (net 18))
@@
   (segment (start 118.415 73.965) (end 116.95 72.5) (width 0.25) (layer F.Cu) (net 18))
   (segment (start 118.415 84.125) (end 118.415 73.965) (width 0.25) (layer F.Cu) (net 18))
+  (segment (start 115.5425 83.0625) (end 115.555 83.075) (width 0.5) (layer F.Cu) (net 19))
+  (segment (start 115.5425 79.68) (end 115.5425 83.0625) (width 0.5) (layer F.Cu) (net 19))
   (segment (start 119.42141 86.4) (end 117.78 84.75859) (width 0.25) (layer F.Cu) (net 19))
   (segment (start 126.26 86.4) (end 119.42141 86.4) (width 0.25) (layer F.Cu) (net 19))
@@
   (segment (start 116.95 82.66) (end 116.315 82.66) (width 0.25) (layer F.Cu) (net 19))
   (segment (start 117.78 83.49) (end 116.95 82.66) (width 0.25) (layer F.Cu) (net 19))
+  (segment (start 115.5425 93.2225) (end 115.555 93.235) (width 0.5) (layer F.Cu) (net 20))
+  (segment (start 115.5425 89.84) (end 115.5425 93.2225) (width 0.5) (layer F.Cu) (net 20))
   (segment (start 126.26 87.05) (end 121.84 87.05) (width 0.25) (layer F.Cu) (net 20))
   (segment (start 119.05 89.84) (end 115.5425 89.84) (width 0.25) (layer F.Cu) (net 20))
