File: KiCad/STM32_Klipper_Expander.sch (KiCad schematic (older format))
At the start: 45 parts, among them J1 USB_B_Micro, J10 Conn_01x01, J11 Conn_01x03, J12 Conn_01x02, J2 Conn_01x04, J4 Conn_01x03, J5 Vin, J6 Screw_Terminal_01x08, J7 Conn_01x02, J8 Conn_01x02, J9 Conn_01x02, Q1 IRLML6344TRPBF, Q2 IRLML6344TRPBF, Q3 IRLML6344TRPBF, Q4 IRLML6344TRPBF, SW2 SW_SPST, U1 STM32F042F6Px, U2 AP2127K-3.3, U3 74LVC1G17

Commit message: file organization
Other:
- moved on the sheet: J4, R6
Changed lines of the file:
@@
 L power:+3V3 #PWR019
 U 1 1 5E23223F
-P 6400 950
-F 0 "#PWR019" H 6400 800 50  0001 C CNN
-F 1 "+3V3" H 6415 1123 50  0000 C CNN
-F 2 "" H 6400 950 50  0001 C CNN
-F 3 "" H 6400 950 50  0001 C CNN
-	1    6400 950
+P 5000 1050
+F 0 "#PWR019" H 5000 900 50  0001 C CNN
+F 1 "+3V3" H 5015 1223 50  0000 C CNN
+F 2 "" H 5000 1050 50  0001 C CNN
+F 3 "" H 5000 1050 50  0001 C CNN
+	1    5000 1050
 	-1   0    0    -1
-$EndComp
-$Comp
-L Connector_Generic:Conn_01x03 J4
-U 1 1 5E23D4FF
-P 7050 1350
-F 0 "J4" H 7130 1392 50  0000 L CNN
-F 1 "Conn_01x03" H 7130 1301 50  0000 L CNN
-F 2 "Connector_PinHeader_2.54mm:PinHeader_1x03_P2.54mm_Vertical" H 7050 1350 50  0001 C CNN
-F 3 "~" H 7050 1350 50  0001 C CNN
-	1    7050 1350
-	1    0    0    -1
 $EndComp
 $Comp
@@
 	1    9500 2000
 	0    -1   -1   0
-$EndComp
-$Comp
-L Device:R R6
-U 1 1 5E3EBE0E
-P 6400 1150
-F 0 "R6" H 6330 1104 50  0000 R CNN
-F 1 "10K" H 6330 1195 50  0000 R CNN
-F 2 "Resistor_SMD:R_0805_2012Metric" V 6330 1150 50  0001 C CNN
-F 3 "~" H 6400 1150 50  0001 C CNN
-F 4 "C17414" H 6400 1150 50  0001 C CNN "LCSC"
-F 5 "RC0805JR-0710KL" H 6330 1204 50  0001 C CNN "MPN"
-F 6 "301010361" H 6330 1204 50  0001 C CNN "SKU"
-	1    6400 1150
-	1    0    0    1
 $EndComp
 Text Label 850  1550 0    50   ~ 0
@@
 VBUS
 Text Label 1950 6100 2    50   ~ 0
-~RESET
-Text Label 6500 1250 0    50   ~ 0
-SWDIO
-Text Label 6500 1350 0    50   ~ 0
-SWDCLK
-Text Label 6500 1450 0    50   ~ 0
 ~RESET
 Text Label 10850 6000 2    50   ~ 0
@@
 	1850 6500 1850 6450
 Wire Wire Line
-	6850 1250 6500 1250
-Wire Wire Line
-	6850 1450 6500 1450
-Wire Wire Line
-	6400 1000 6400 950
-Wire Wire Line
-	6400 1350 6400 1300
-Wire Wire Line
-	6400 1350 6850 1350
+	5000 1100 5000 1050
 Wire Wire Line
 	10500 5800 10850 5800
@@
 Connection ~ 7750 5700
 Connection ~ 7750 5550
+Wire Wire Line
+	5000 1450 5450 1450
+Wire Wire Line
+	5000 1450 5000 1400
+Wire Wire Line
+	5450 1550 5100 1550
+Wire Wire Line
+	5450 1350 5100 1350
+Text Label 5100 1550 0    50   ~ 0
+~RESET
+Text Label 5100 1450 0    50   ~ 0
+SWDCLK
+Text Label 5100 1350 0    50   ~ 0
+SWDIO
+$Comp
+L Device:R R6
+U 1 1 5E3EBE0E
+P 5000 1250
+F 0 "R6" H 4930 1204 50  0000 R CNN
+F 1 "10K" H 4930 1295 50  0000 R CNN
+F 2 "Resistor_SMD:R_0805_2012Metric" V 4930 1250 50  0001 C CNN
+F 3 "~" H 5000 1250 50  0001 C CNN
+F 4 "C17414" H 5000 1250 50  0001 C CNN "LCSC"
+F 5 "RC0805JR-0710KL" H 4930 1304 50  0001 C CNN "MPN"
+F 6 "301010361" H 4930 1304 50  0001 C CNN "SKU"
+	1    5000 1250
+	1    0    0    1
+$EndComp
+$Comp
+L Connector_Generic:Conn_01x03 J4
+U 1 1 5E23D4FF
+P 5650 1450
+F 0 "J4" H 5730 1492 50  0000 L CNN
+F 1 "Conn_01x03" H 5730 1401 50  0000 L CNN
+F 2 "Connector_PinHeader_2.54mm:PinHeader_1x03_P2.54mm_Vertical" H 5650 1450 50  0001 C CNN
+F 3 "~" H 5650 1450 50  0001 C CNN
+	1    5650 1450
+	1    0    0    -1
+$EndComp
 $EndSCHEMATC

Commit message: Klipper Expander V2
Update to Klipper Expander that adds status LED's to the 4 mosfet outputs, 5V rail, and Vin rail.
Also changed 2 capacitors to use the same 4.7uF that are already present lowering the unique part count.
Parts:
- removed R16, R17: 10K, Resistor_SMD:R_0805_2012Metric, symbol Device:R
- added D2, D3, D4, D5, D6, D7: LED, KlipperExpander:LED_0805_2012Metric, symbol KlipperExpander:LED
- added R15, R16, R17, R18, R19, R20, R22: 4.7K, KlipperExpander:R_0805_2012Metric, symbol KlipperExpander:R
- added R21: 1K, KlipperExpander:R_0805_2012Metric, symbol KlipperExpander:R
- C1, C2, C3, C4: footprint Capacitor_SMD:C_0805_2012Metric -> KlipperExpander:C_0805_2012Metric; symbol Device:C -> KlipperExpander:C
- C5, C6: value 10uF -> 4.7uF; footprint Capacitor_SMD:C_0805_2012Metric -> KlipperExpander:C_0805_2012Metric; symbol Device:C -> KlipperExpander:C; LCSC C15850 -> C1779; MPN CC0805ZKY5V6BB106 -> CC0805KKX5R8BB475; SKU 302010158 -> 302010146
- D1: footprint LED_SMD:LED_0805_2012Metric -> KlipperExpander:LED_0805_2012Metric; symbol Device:LED -> KlipperExpander:LED
- F1: footprint TRA_KiCad_Footprints:3544-2_FuseHolder -> KlipperExpander:3544-2_FuseHolder; symbol Device:Fuse -> KlipperExpander:Fuse
- H1, H2: footprint MountingHole:MountingHole_3.2mm_M3 -> KlipperExpander:MountingHole_3.2mm_M3
- J1: footprint TRA_KiCad_Footprints:Molex-105017-0001-USBMicroB -> KlipperExpander:Molex-105017-0001-USBMicroB; symbol Connector:USB_B_Micro -> KlipperExpander:USB_B_Micro
- J10: footprint Connector_PinHeader_2.54mm:PinHeader_1x01_P2.54mm_Vertical -> KlipperExpander:PinHeader_1x01_P2.54mm_Vertical; symbol Connector_Generic:Conn_01x01 -> KlipperExpander:Conn_01x01
- J11, J4: footprint Connector_PinHeader_2.54mm:PinHeader_1x03_P2.54mm_Vertical -> KlipperExpander:PinHeader_1x03_P2.54mm_Vertical; symbol Connector_Generic:Conn_01x03 -> KlipperExpander:Conn_01x03
- J12: value Conn_01x02 -> Conn_01x03; footprint Connector_PinHeader_2.54mm:PinHeader_1x02_P2.54mm_Vertical -> KlipperExpander:PinHeader_1x03_P2.54mm_Vertical; symbol Connector_Generic:Conn_01x02 -> KlipperExpander:Conn_01x03
- J2: footprint Connector_PinHeader_2.54mm:PinHeader_1x04_P2.54mm_Vertical -> KlipperExpander:PinHeader_1x04_P2.54mm_Vertical; symbol Connector_Generic:Conn_01x04 -> KlipperExpander:Conn_01x04
- J5: footprint TRA_KiCad_Footprints:1x02_ScrewTerminal_Phoenix -> KlipperExpander:1x02_ScrewTerminal_Phoenix; symbol Connector:Screw_Terminal_01x02 -> KlipperExpander:Screw_Terminal_01x02
- J6: footprint TRA_KiCad_Footprints:TerminalBlock_Phoenix_MKDS-1,5-8-5.08_1x08_P5.08mm_Horizontal -> KlipperExpander:1x08_ScrewTerminal_Phoenix; symbol Connector:Screw_Terminal_01x08 -> KlipperExpander:Screw_Terminal_01x08
- J7: footprint Connector_PinHeader_2.54mm:PinHeader_1x02_P2.54mm_Vertical -> KlipperExpander:PinHeader_1x02_P2.54mm_Vertical; symbol Connector_Generic:Conn_01x02 -> KlipperExpander:Conn_01x02
- J8, J9: footprint Connector_JST:JST_XH_B02B-XH-A_1x02_P2.50mm_Vertical -> KlipperExpander:PinHeader_1x02_P2.54mm_Vertical; symbol Connector_Generic:Conn_01x02 -> KlipperExpander:Conn_01x02
- Q1, Q2, Q3, Q4: footprint Package_TO_SOT_SMD:SOT-23 -> KlipperExpander:SOT-23; symbol dk_Transistors-FETs-MOSFETs-Single:IRLML6344TRPBF -> KlipperExpander:IRLML6344TRPBF
- R1, R10, R11, R12, R13, R14, R2, R3, R4, R5, R6, R7, R8, R9: footprint Resistor_SMD:R_0805_2012Metric -> KlipperExpander:R_0805_2012Metric; symbol Device:R -> KlipperExpander:R
- SW2: footprint TRA_KiCad_Footprints:2PinTactileButton -> KlipperExpander:2PinTactileButton; symbol Switch:SW_SPST -> KlipperExpander:SW_SPST
- U1: footprint Package_SO:TSSOP-20_4.4x6.5mm_P0.65mm -> KlipperExpander:TSSOP-20_4.4x6.5mm_P0.65mm; symbol MCU_ST_STM32F0:STM32F042F6Px -> KlipperExpander:STM32F042F6Px
- U2: footprint Package_TO_SOT_SMD:SOT-23-5 -> KlipperExpander:SOT-23-5; symbol Regulator_Linear:AP2127K-3.3 -> KlipperExpander:AP2127K-3.3
- U3: footprint Package_TO_SOT_SMD:SOT-353_SC-70-5 -> KlipperExpander:SOT-753; symbol 74xGxx:74LVC1G17 -> KlipperExpander:74LVC1G17; LCSC C124293 -> C6076; MPN 74LVC1G17SE-7 -> (none)
Connections:
- net +3V3: now also J12.2 (Pin_2), R16.2, R17.2
- net GND: now also J12.3 (Pin_3), D6.1 (K), D7.1 (K); no longer J12.2 (Pin_2)
- net Mosfet0: now also D2.1 (K)
- net Mosfet1: now also D3.1 (K)
- net Mosfet2: now also D4.1 (K)
- net Mosfet3: now also D5.1 (K)
- net T0: now also R16.1
- net T1: now also R17.1
- net VCC: now also R21.2
- net Vin: now also R15.1, R18.1, R19.1, R20.1, R22.2
- new net: D2.2 (A), R15.2
- new net: D5.2 (A), R20.2
- new net: D4.2 (A), R19.2
- new net: D3.2 (A), R18.2
- new net: D7.2 (A), R22.1
- new net: D6.2 (A), R21.1
Other:
- moved on the sheet: Q4, R10, R14
